File: _autosave-macropad.kicad_pcb (KiCad board)
At the start: 4 copper layers, 33 parts, among them M1 1U

Commit message: pcb
Routing:
- net (no net): track 1484.7 -> 1499.6 mm
Changed lines of the file:
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@@
   )
   (segment (start 110.180088 75.845384) (end 108.933912 75.845384) (width 0.15) (layer "F.Cu") (net 0))
-  (segment (start 162.258021 65.87344) (end 153.687931 65.87344) (width 0.15) (layer "F.Cu") (net 0))
   (segment (start 110.180088 51.873164) (end 110.180088 75.845384) (width 0.15) (layer "F.Cu") (net 0))
-  (segment (start 153.687931 71.10774) (end 153.687931 83.585698) (width 0.15) (layer "F.Cu") (net 0))
+  (segment (start 153.687931 83.65344) (end 162.258021 83.65344) (width 0.15) (layer "F.Cu") (net 0))
+  (segment (start 142.200318 71.10774) (end 142.200318 75.598978) (width 0.15) (layer "F.Cu") (net 0))
   (segment (start 167.338021 83.65344) (end 172.392342 83.65344) (width 0.15) (layer "F.Cu") (net 0))
   (segment (start 164.798021 68.744057) (end 164.795744 68.746334) (width 0) (layer "F.Cu") (net 0))
-  (segment (start 153.687931 65.87344) (end 153.687931 71.10774) (width 0.15) (layer "F.Cu") (net 0))
   (segment (start 168.239789 65.908822) (end 172.38911 65.908822) (width 0.15) (layer "F.Cu") (net 0))
   (segment (start 153.687931 71.10774) (end 153.645856 71.149814) (width 0) (layer "F.Cu") (net 0))
+  (segment (start 142.200318 75.598978) (end 141.953912 75.845384) (width 0) (layer "F.Cu") (net 0))
+  (segment (start 153.687931 71.10774) (end 142.200318 71.10774) (width 0.15) (layer "F.Cu") (net 0))
+  (segment (start 153.687931 65.87344) (end 153.687931 83.65344) (width 0.15) (layer "F.Cu") (net 0))
   (segment (start 172.392342 51.873164) (end 110.180088 51.873164) (width 0.15) (layer "F.Cu") (net 0))
-  (segment (start 153.687931 83.585698) (end 153.755673 83.65344) (width 0.15) (layer "F.Cu") (net 0))
   (segment (start 172.392342 51.873164) (end 172.392342 83.65344) (width 0.15) (layer "F.Cu") (net 0))
-  (segment (start 153.755673 83.65344) (end 162.258021 83.65344) (width 0.15) (layer "F.Cu") (net 0))
+  (segment (start 162.258021 65.87344) (end 153.687931 65.87344) (width 0.15) (layer "F.Cu") (net 0))
   (via (at 120.89652 136.542477) (size 0.8) (drill 0.4) (layers "F.Cu" "B.Cu") (free) (net 0))
   (via (at 163.530752 90.958028) (size 0.8) (drill 0.4) (layers "F.Cu" "B.Cu") (free) (net 0))
@@
   (segment (start 105.085816 85.7079) (end 108.213227 88.835311) (width 0.25) (layer "In2.Cu") (net 0))
   (segment (start 108.213227 88.835311) (end 116.147391 88.835311) (width 0.25) (layer "In2.Cu") (net 0))
+  (segment (start 159.726163 87.067807) (end 159.726163 85.696007) (width 0.15) (layer "B.Cu") (net 0))
   (segment (start 156.529446 133.828548) (end 156.529446 134.768356) (width 0.15) (layer "B.Cu") (net 0))
   (segment (start 106.776639 105.617632) (end 103.786375 105.617632) (width 0.15) (layer "B.Cu") (net 0))
-  (segment (start 118.430127 95.01034) (end 118.430127 91.967807) (width 0.15) (layer "B.Cu") (net 0))
   (segment (start 126.713912 75.845384) (end 126.713912 81.984022) (width 0.15) (layer "B.Cu") (net 0))
+  (segment (start 118.430127 94.479199) (end 118.430127 91.967807) (width 0.15) (layer "B.Cu") (net 0))
   (segment (start 144.78 123.66471) (end 144.958845 123.843555) (width 0) (layer "B.Cu") (net 0))
   (segment (start 125.73 115.57) (end 125.73 123.726987) (width 0.15) (layer "B.Cu") (net 0))
   (segment (start 119.093912 79.278369) (end 102.042699 96.329582) (width 0.15) (layer "B.Cu") (net 0))
+  (segment (start 129.739569 94.479199) (end 118.430127 94.479199) (width 0.15) (layer "B.Cu") (net 0))
   (segment (start 144.78 96.52) (end 144.78 103.358404) (width 0.15) (layer "B.Cu") (net 0))
   (segment (start 164.798021 68.973338) (end 144.493912 68.973338) (width 0.15) (layer "B.Cu") (net 0))
   (segment (start 154.08646 128.015631) (end 154.999377 128.928548) (width 0.15) (layer "B.Cu") (net 0))
   (segment (start 147.542214 131.935619) (end 136.151788 131.935619) (width 0.15) (layer "B.Cu") (net 0))
-  (segment (start 136.878124 85.411651) (end 129.739569 92.550206) (width 0.15) (layer "B.Cu") (net 0))
   (segment (start 106.68 123.777299) (end 106.776639 123.873938) (width 0) (layer "B.Cu") (net 0))
   (segment (start 142.225102 58.405102) (end 142.24 58.42) (width 0) (layer "B.Cu") (net 0))
@@
   (segment (start 163.83 115.57) (end 163.83 123.853842) (width 0.15) (layer "B.Cu") (net 0))
   (segment (start 132.47228 135.615127) (end 125.785701 128.928548) (width 0.15) (layer "B.Cu") (net 0))
+  (segment (start 159.726163 85.696007) (end 136.593768 85.696007) (width 0.15) (layer "B.Cu") (net 0))
   (segment (start 92.535848 91.747905) (end 92.497927 91.785826) (width 0) (layer "B.Cu") (net 0))
   (segment (start 174.139218 128.928548) (end 159.729446 128.928548) (width 0.15) (layer "B.Cu") (net 0))
   (segment (start 123.106795 91.967807) (end 124.566302 90.5083) (width 0.15) (layer "B.Cu") (net 0))
   (segment (start 102.950244 96.650942) (end 102.950244 125.923938) (width 0.15) (layer "B.Cu") (net 0))
+  (segment (start 136.593768 85.696007) (end 129.739569 92.550206) (width 0.15) (layer "B.Cu") (net 0))
   (segment (start 125.73 103.420681) (end 125.876951 103.567632) (width 0) (layer "B.Cu") (net 0))
   (segment (start 163.850096 125.923938) (end 163.85655 125.930392) (width 0) (layer "B.Cu") (net 0))
@@
   (segment (start 163.966788 103.509787) (end 163.83 103.372999) (width 0.25) (layer "B.Cu") (net 0))
   (segment (start 164.798021 65.87344) (end 164.798021 68.973338) (width 0.15) (layer "B.Cu") (net 0))
+  (segment (start 129.739569 92.550206) (end 129.739569 94.479199) (width 0.15) (layer "B.Cu") (net 0))
   (segment (start 163.83 103.547536) (end 163.85655 103.574086) (width 0) (layer "B.Cu") (net 0))
   (segment (start 172.137759 91.967807) (end 172.233944 92.063992) (width 0.15) (layer "B.Cu") (net 0))
-  (segment (start 129.739569 95.01034) (end 118.430127 95.01034) (width 0.15) (layer "B.Cu") (net 0))
   (segment (start 125.73 96.52) (end 125.73 103.420681) (width 0.15) (layer "B.Cu") (net 0))
   (segment (start 147.033912 84.898512) (end 147.033912 75.845384) (width 0.15) (layer "B.Cu") (net 0))
@@
   (segment (start 124.173912 76.681471) (end 124.173912 75.845384) (width 0.15) (layer "B.Cu") (net 0))
   (segment (start 159.729446 135.378785) (end 159.729446 133.828548) (width 0.15) (layer "B.Cu") (net 0))
-  (segment (start 159.726163 85.411651) (end 136.878124 85.411651) (width 0.15) (layer "B.Cu") (net 0))
   (segment (start 106.785526 103.457437) (end 106.68 103.351911) (width 0.25) (layer "B.Cu") (net 0))
   (segment (start 106.783093 105.624086) (end 106.776639 105.617632) (width 0) (layer "B.Cu") (net 0))
@@
   (segment (start 162.520973 91.967807) (end 163.530752 90.958028) (width 0.15) (layer "B.Cu") (net 0))
   (segment (start 121.633912 77.967274) (end 102.950244 96.650942) (width 0.15) (layer "B.Cu") (net 0))
-  (segment (start 129.739569 92.550206) (end 129.739569 95.01034) (width 0.15) (layer "B.Cu") (net 0))
   (segment (start 163.83 142.627221) (end 163.85655 142.653771) (width 0) (layer "B.Cu") (net 0))
   (segment (start 121.633912 75.845384) (end 121.633912 77.967274) (width 0.15) (layer "B.Cu") (net 0))
@@
   (segment (start 164.798021 84.495073) (end 164.798021 84.898512) (width 0.15) (layer "B.Cu") (net 0))
   (segment (start 126.713912 81.984022) (end 121.630127 87.067807) (width 0.15) (layer "B.Cu") (net 0))
-  (segment (start 159.726163 87.067807) (end 159.726163 85.411651) (width 0.15) (layer "B.Cu") (net 0))
   (segment (start 154.140428 87.054388) (end 156.512744 87.054388) (width 0.15) (layer "B.Cu") (net 0))
   (segment (start 106.68 115.57) (end 106.68 123.777299) (width 0.15) (layer "B.Cu") (net 0))
